Commit message: controller load success

File: ppr_description/urdf/gtrobot_arm/ur.transmission.xacro (robot description, xacro)
@@ -2,61 +2,63 @@
 <robot xmlns:xacro="http://wiki.ros.org/xacro">
   <xacro:macro name="gtrobot_arm_transmission" params="prefix hw_interface">
-    <transmission name="${prefix}shoulder_pan_trans">
+    <xacro:arg name="poineer_arm_prefix" default="poineer::gtrobot_arm::"/>
+    <!-- <xacro:property name="poineer_arm_prefix" value="poineer::"/> -->
+    <transmission name="$(arg poineer_arm_prefix)${prefix}shoulder_pan_trans">
       <type>transmission_interface/SimpleTransmission</type>
-      <joint name="${prefix}shoulder_pan_joint">
+      <joint name="$(arg poineer_arm_prefix)${prefix}shoulder_pan_joint">
         <hardwareInterface>${hw_interface}</hardwareInterface>
         <hardwareInterface>hardware_interface/VelocityJointInterface</hardwareInterface>
       </joint>
-      <actuator name="${prefix}shoulder_pan_motor">
+      <actuator name="$(arg poineer_arm_prefix)${prefix}shoulder_pan_motor">
         <mechanicalReduction>1</mechanicalReduction>
       </actuator>
     </transmission>
-    <transmission name="${prefix}shoulder_lift_trans">
+    <transmission name="$(arg poineer_arm_prefix)${prefix}shoulder_lift_trans">
       <type>transmission_interface/SimpleTransmission</type>
-      <joint name="${prefix}shoulder_lift_joint">
+      <joint name="$(arg poineer_arm_prefix)${prefix}shoulder_lift_joint">
         <hardwareInterface>${hw_interface}</hardwareInterface>
         <hardwareInterface>hardware_interface/VelocityJointInterface</hardwareInterface>
       </joint>
-      <actuator name="${prefix}shoulder_lift_motor">
+      <actuator name="$(arg poineer_arm_prefix)${prefix}shoulder_lift_motor">
         <mechanicalReduction>1</mechanicalReduction>
       </actuator>
     </transmission>
-    <transmission name="${prefix}elbow_trans">
+    <transmission name="$(arg poineer_arm_prefix)${prefix}elbow_trans">
       <type>transmission_interface/SimpleTransmission</type>
-      <joint name="${prefix}elbow_joint">
+      <joint name="$(arg poineer_arm_prefix)${prefix}elbow_joint">
         <hardwareInterface>${hw_interface}</hardwareInterface>
         <hardwareInterface>hardware_interface/VelocityJointInterface</hardwareInterface>
       </joint>
-      <actuator name="${prefix}elbow_motor">
+      <actuator name="$(arg poineer_arm_prefix)${prefix}elbow_motor">
         <mechanicalReduction>1</mechanicalReduction>
       </actuator>
     </transmission>
-    <transmission name="${prefix}wrist_1_trans">
+    <transmission name="$(arg poineer_arm_prefix)${prefix}wrist_1_trans">
       <type>transmission_interface/SimpleTransmission</type>
-      <joint name="${prefix}wrist_1_joint">
+      <joint name="$(arg poineer_arm_prefix)${prefix}wrist_1_joint">
         <hardwareInterface>${hw_interface}</hardwareInterface>
         <hardwareInterface>hardware_interface/VelocityJointInterface</hardwareInterface>
       </joint>
-      <actuator name="${prefix}wrist_1_motor">
+      <actuator name="$(arg poineer_arm_prefix)${prefix}wrist_1_motor">
         <mechanicalReduction>1</mechanicalReduction>
       </actuator>
     </transmission>
-    <transmission name="${prefix}wrist_2_trans">
+    <transmission name="$(arg poineer_arm_prefix)${prefix}wrist_2_trans">
       <type>transmission_interface/SimpleTransmission</type>
-      <joint name="${prefix}wrist_2_joint">
+      <joint name="$(arg poineer_arm_prefix)${prefix}wrist_2_joint">
         <hardwareInterface>${hw_interface}</hardwareInterface>
         <hardwareInterface>hardware_interface/VelocityJointInterface</hardwareInterface>
       </joint>
-      <actuator name="${prefix}wrist_2_motor">
+      <actuator name="$(arg poineer_arm_prefix)${prefix}wrist_2_motor">
         <mechanicalReduction>1</mechanicalReduction>
       </actuator>
     </transmission>
-    <transmission name="${prefix}wrist_3_trans">
+    <transmission name="$(arg poineer_arm_prefix)${prefix}wrist_3_trans">
       <type>transmission_interface/SimpleTransmission</type>
-      <joint name="${prefix}wrist_3_joint">
+      <joint name="$(arg poineer_arm_prefix)${prefix}wrist_3_joint">
         <hardwareInterface>${hw_interface}</hardwareInterface>
         <hardwareInterface>hardware_interface/VelocityJointInterface</hardwareInterface>
       </joint>
-      <actuator name="${prefix}wrist_3_motor">
+      <actuator name="$(arg poineer_arm_prefix)${prefix}wrist_3_motor">
         <mechanicalReduction>1</mechanicalReduction>
       </actuator>

File: ppr_description/urdf/gtrobot_base/base.transmission.xacro (robot description, xacro)
@@ -6,13 +6,14 @@
   <xacro:property name="wheel_mechanical_reduction" value="${624/35 * 80/18}" />
   <xacro:property name="caster_mechanical_reduction" value="${624/35 * 80/18}" />
+  <xacro:arg name="poineer_prefix" default="poineer::gtrobot_base::"/>
   <!--  Wheel transmission   -->
   <xacro:macro name="wheel_transmission" params="parent">
-    <transmission name="${parent}_wheel_trans">
+    <transmission name="$(arg poineer_prefix)${parent}_wheel_trans">
       <type>transmission_interface/SimpleTransmission</type>
-      <actuator name="${parent}_wheel_motor" >
+      <actuator name="$(arg poineer_prefix)${parent}_wheel_motor" >
         <hardwareInterface>hardware_interface/VelocityJointInterface</hardwareInterface>
         <mechanicalReduction>${wheel_mechanical_reduction}</mechanicalReduction>
       </actuator>
-      <joint name="${parent}_wheel_joint" >
+      <joint name="$(arg poineer_prefix)${parent}_wheel_joint" >
         <hardwareInterface>hardware_interface/VelocityJointInterface</hardwareInterface>
       </joint>
@@ -21,11 +22,11 @@
   <!-- Caster transmission   -->
   <xacro:macro name="caster_transmission" params="suffix">
-    <transmission name="${suffix}_rotation_trans">
+    <transmission name="$(arg poineer_prefix)${suffix}_rotation_trans">
       <type>transmission_interface/SimpleTransmission</type>
-      <actuator name="${suffix}_rotation_motor">
+      <actuator name="$(arg poineer_prefix)${suffix}_rotation_motor">
         <hardwareInterface>hardware_interface/VelocityJointInterface</hardwareInterface>
         <mechanicalReduction>${caster_mechanical_reduction}</mechanicalReduction>
       </actuator>
-      <joint name="${suffix}_rotation_joint" >
+      <joint name="$(arg poineer_prefix)${suffix}_rotation_joint" >
         <hardwareInterface>hardware_interface/VelocityJointInterface</hardwareInterface>
       </joint>
@@ -36,8 +37,8 @@
     <transmission name="tran_x">
       <type>transmission_interface/SimpleTransmission</type>
-      <joint name="x_axis_joint">
+      <joint name="$(arg poineer_prefix)x_axis_joint">
         <hardwareInterface>${hw_interface}</hardwareInterface>
       </joint>
-      <actuator name="motor_x">
+      <actuator name="$(arg poineer_prefix)motor_x">
         <hardwareInterface>${hw_interface}</hardwareInterface>
         <mechanicalReduction>1</mechanicalReduction>
@@ -47,8 +48,8 @@
     <transmission name="tran_y">
       <type>transmission_interface/SimpleTransmission</type>
-      <joint name="y_axis_joint">
+      <joint name="$(arg poineer_prefix)y_axis_joint">
         <hardwareInterface>${hw_interface}</hardwareInterface>
       </joint>
-      <actuator name="motor_y">
+      <actuator name="$(arg poineer_prefix)motor_y">
         <hardwareInterface>${hw_interface}</hardwareInterface>
         <mechanicalReduction>1</mechanicalReduction>
@@ -58,8 +59,8 @@
     <transmission name="trans_rotate">
       <type>transmission_interface/SimpleTransmission</type>
-      <joint name="rotate_axis_joint">
+      <joint name="$(arg poineer_prefix)rotate_axis_joint">
         <hardwareInterface>${hw_interface}</hardwareInterface>
       </joint>
-      <actuator name="motor_rotate" >
+      <actuator name="$(arg poineer_prefix)motor_rotate" >
         <hardwareInterface>${hw_interface}</hardwareInterface>
         <mechanicalReduction>${caster_mechanical_reduction}</mechanicalReduction>

File: ppr_description/urdf/ppr.xacro (robot description, xacro)
@@ -107,10 +107,10 @@
     <joint name="motor4" type="revolute">
         <parent link="link2"/>
-        <child link="upper_link"/>
+        <child link="ppr_upper_link"/>
         <limit lower="-3.14" upper="3.14" effort="100.0" velocity="1.7"/>
         <origin xyz="0 0 ${height2}" rpy="0.0 0.0 0"/>
         <axis xyz="1 0 0"/>
     </joint>
-    <link name="upper_link">
+    <link name="ppr_upper_link">
          <collision>
             <origin xyz="0 ${width1} 0" rpy="0.0 0.0 0.0"/>
@@ -261,7 +261,8 @@
     </joint>
     <link name="camera_link_optical"/> -->
+<!--
     <transmission name="tran1">
         <type>transmission_interface/SimpleTransmission</type>
-        <joint name="motor1">
+        <joint name="poineer::motor1">
             <hardwareInterface>hardware_interface/EffortJointInterface</hardwareInterface>
         </joint>
@@ -273,5 +274,5 @@
     <transmission name="tran2">
         <type>transmission_interface/SimpleTransmission</type>
-        <joint name="motor2">
+        <joint name="poineer::motor2">
             <hardwareInterface>hardware_interface/EffortJointInterface</hardwareInterface>
         </joint>
@@ -283,5 +284,5 @@
     <transmission name="tran3">
         <type>transmission_interface/SimpleTransmission</type>
-        <joint name="upper_joint">
+        <joint name="poineer::motor3">
             <hardwareInterface>hardware_interface/EffortJointInterface</hardwareInterface>
         </joint>
@@ -290,4 +291,4 @@
             <mechanicalReduction>1</mechanicalReduction>
         </actuator>
-    </transmission>
+    </transmission> -->
 </robot>
