Commit message: Update

File: ppr_description/urdf/gtrobot.urdf.xacro (robot description, xacro)
@@ -1,5 +1,5 @@
 <?xml version="1.0"?>
 <robot xmlns:xacro="http://wiki.ros.org/xacro"
-       name="gtrobot" >
+       name="poineer" >
   <!-- The following xacro:included files set up definitions of parts of the robot body -->
   <!-- misc common stuff? controller manager-->
@@ -93,65 +93,4 @@
     <xacro:rplidar prefix="lidar"/>
   </xacro:if>
-  <!-- infrared ray -->
-  <xacro:if value="$(arg infrared_ray_enabled)">
-    <joint name="infrared_ray_joint" type="fixed">
-        <origin xyz="${infrared_ray_offset_x} ${infrared_ray_offset_y} ${infrared_ray_offset_z}" rpy="${pi/2} 0 0" />
-        <parent link="arm_ee_link"/>
-        <child link="infrared_ray_link"/>
-    </joint>
-    <xacro:infrared_ray prefix="infrared_ray"/>
-  </xacro:if>
-  <!--Stereo Camera Joint-->
-  <xacro:if value="$(arg zed_enabled)">
-    <joint name="stereo_joint" type="fixed">
-      <parent link="${zed_base_parent}"/>
-      <child link="base_stereo"/>
-      <origin xyz="${zed_offset_x} ${zed_offset_y} ${zed_offset_z}"
-              rpy="${zed_offset_roll} ${zed_offset_pitch} ${zed_offset_yaw}"/>
-    </joint>
-    <link name="base_stereo">
-      <visual>
-        <origin xyz="0 0 0" rpy="0 0 0"/>
-        <geometry>
-          <mesh filename="package://ppr_description/meshes/sensors/ZED.stl" />
-        </geometry>
-        <material name="dark"/>
-      </visual>
-      <xacro:cuboid_inertial length="0.16" weight="0.04" hight="0.04" mass="0.00000001">
-        <origin xyz="0.0 0.0 0.0" rpy="0 0 0" />
-      </xacro:cuboid_inertial>
-    </link>
-    <xacro:stereo_camera_v0 parent="base_stereo" name="stereo" focal_length="700.065972" hfov="84.8725" image_width="1280" image_height="720" >
-        <origin xyz="0 0 0.0" rpy="0.0   0.0   0.0" />
-    </xacro:stereo_camera_v0>
-  </xacro:if>
-  <!--Stereo Camera Virtual Joint for Collision Avoidance-->
-  <!-- <joint name="left_stereo_virtual_joint" type="fixed">
-    <parent link="arm_ee_link"/>
-    <child link="collision_virtual_ee_link"/>
-    <origin xyz="0.5 0 0"
-            rpy="${pi/2} 0 ${pi/2}"/>
-  </joint>
-  <link name="collision_virtual_ee_link">
-    <visual>
-      <origin xyz="0 0 0" rpy="0 0 0"/>
-      <geometry>
-        <cylinder radius="0.0001" length="0.0001" />
-      </geometry>
-      <material name="dark"/>
-    </visual>
-    <xacro:cylinder_inertial length="0.05" radius="0.1" mass="0.00000001">
-      <origin xyz="0.0 0.0 0.0" rpy="0 0 0" />
-    </xacro:cylinder_inertial>
-  </link> -->
-  <!-- imu -->
-  <xacro:if value="$(arg imu_enabled)">
-    <joint name="imu_joint" type="fixed">
-        <origin xyz="${imu_offset_x} ${imu_offset_y} ${imu_offset_z}" rpy="${imu_offset_roll} ${imu_offset_pitch} ${imu_offset_yaw}" />
-        <parent link="${imu_base_parent}"/>
-        <child link="imu_link"/>
-    </joint>
-    <xacro:imu prefix="imu"/>
-  </xacro:if>
   <!-- ground truth for arm_wrist_3_link -->
   <gazebo>

File: ppr_description/urdf/gtrobot_base_only.urdf.xacro (robot description, xacro)
@@ -1,5 +1,5 @@
 <?xml version="1.0"?>
 <robot xmlns:xacro="http://wiki.ros.org/xacro"
-       name="gtrobot" >
+       name="poineer" >
   <!-- The following xacro:included files set up definitions of parts of the robot body -->
   <!-- misc common stuff? controller manager-->

Commit message: merge urdf ppr to gtrobot

File: ppr_description/urdf/gtrobot.urdf.xacro (robot description, xacro)
@@ -50,4 +50,14 @@
     <xacro:property name="zed_offset_yaw" value="${-pi/2}" />
   </xacro:unless>
+  <!-- PARABOT -->
+  <xacro:arg name="parabot_enabled" default="true"/>
+  <xacro:if value="$(arg parabot_enabled)">
+    <xacro:include filename="$(find ppr_description)/urdf/ppr.xacro"/>
+    <joint name="parabot_fixed" type="fixed">
+      <parent link="$(arg ur_prefix)wrist_3_link"/>
+      <child link="link1"/>
+      <origin xyz="0.0 0.0 0.0" rpy="0.0 0.0 0.0"/>
+    </joint>
+  </xacro:if>
   <!-- IMU -->
   <xacro:include filename="$(find ppr_description)/urdf/sensors/imu_gazebo.xacro" />

File: ppr_description/urdf/ppr.xacro (robot description, xacro)
@@ -13,10 +13,10 @@
     <xacro:include filename="$(find ppr_description)/urdf/ppr.gazebo"/>
     <xacro:include filename="$(find ppr_description)/urdf/materials.xacro"/>
-    <link name="world"/>
+    <!-- <link name="world"/>
     <joint name="fixed" type="fixed">
         <parent link="world"/>
         <child link="link1"/>
         <origin xyz="0.0 0.0 0.0" rpy="0.0 0.0 0.0"/>
-    </joint>
+    </joint> -->
     <link name="link1">
         <collision>

Commit message: debug controller for gazebo

File: ppr_description/urdf/gtrobot.urdf.xacro (robot description, xacro)
@@ -5,5 +5,5 @@
   <!-- misc common stuff? controller manager-->
   <!--<xacro:include filename="$(find ppr_description)/urdf/common.xacro" />-->
-  <xacro:include filename="$(find ppr_description)/urdf/common.gazebo.xacro" />
+  <!-- <xacro:include filename="$(find ppr_description)/urdf/common.gazebo.xacro" /> -->
   <!-- gtrobot base -->
   <xacro:include filename="$(find ppr_description)/urdf/gtrobot_base/base.urdf.xacro" />

File: ppr_description/urdf/gtrobot_arm/ur.transmission.xacro (robot description, xacro)
@@ -3,10 +3,8 @@
   <xacro:macro name="gtrobot_arm_transmission" params="prefix hw_interface">
     <xacro:arg name="poineer_arm_prefix" default="poineer::gtrobot_arm::"/>
-    <!-- <xacro:property name="poineer_arm_prefix" value="poineer::"/> -->
     <transmission name="$(arg poineer_arm_prefix)${prefix}shoulder_pan_trans">
       <type>transmission_interface/SimpleTransmission</type>
       <joint name="$(arg poineer_arm_prefix)${prefix}shoulder_pan_joint">
         <hardwareInterface>${hw_interface}</hardwareInterface>
-        <hardwareInterface>hardware_interface/VelocityJointInterface</hardwareInterface>
       </joint>
       <actuator name="$(arg poineer_arm_prefix)${prefix}shoulder_pan_motor">
@@ -18,5 +16,4 @@
       <joint name="$(arg poineer_arm_prefix)${prefix}shoulder_lift_joint">
         <hardwareInterface>${hw_interface}</hardwareInterface>
-        <hardwareInterface>hardware_interface/VelocityJointInterface</hardwareInterface>
       </joint>
       <actuator name="$(arg poineer_arm_prefix)${prefix}shoulder_lift_motor">
@@ -28,5 +25,4 @@
       <joint name="$(arg poineer_arm_prefix)${prefix}elbow_joint">
         <hardwareInterface>${hw_interface}</hardwareInterface>
-        <hardwareInterface>hardware_interface/VelocityJointInterface</hardwareInterface>
       </joint>
       <actuator name="$(arg poineer_arm_prefix)${prefix}elbow_motor">
@@ -38,5 +34,4 @@
       <joint name="$(arg poineer_arm_prefix)${prefix}wrist_1_joint">
         <hardwareInterface>${hw_interface}</hardwareInterface>
-        <hardwareInterface>hardware_interface/VelocityJointInterface</hardwareInterface>
       </joint>
       <actuator name="$(arg poineer_arm_prefix)${prefix}wrist_1_motor">
@@ -48,5 +43,4 @@
       <joint name="$(arg poineer_arm_prefix)${prefix}wrist_2_joint">
         <hardwareInterface>${hw_interface}</hardwareInterface>
-        <hardwareInterface>hardware_interface/VelocityJointInterface</hardwareInterface>
       </joint>
       <actuator name="$(arg poineer_arm_prefix)${prefix}wrist_2_motor">
@@ -58,5 +52,4 @@
       <joint name="$(arg poineer_arm_prefix)${prefix}wrist_3_joint">
         <hardwareInterface>${hw_interface}</hardwareInterface>
-        <hardwareInterface>hardware_interface/VelocityJointInterface</hardwareInterface>
       </joint>
       <actuator name="$(arg poineer_arm_prefix)${prefix}wrist_3_motor">

File: ppr_description/urdf/gtrobot_arm/ur5_robot.urdf.xacro (robot description, xacro)
@@ -8,5 +8,5 @@
   <xacro:arg name="urbase_parent" default="upper_link"/>
   <!-- common stuff -->
-  <xacro:include filename="$(find ppr_description)/urdf/common.gazebo.xacro" />
+  <!-- <xacro:include filename="$(find ppr_description)/urdf/common.gazebo.xacro" /> -->
   <!-- ur5 -->
   <xacro:include filename="$(find ppr_description)/urdf/gtrobot_arm/ur5.urdf.xacro" />

Commit message: add multiple functions

File: ppr_description/urdf/gtrobot.urdf.xacro (robot description, xacro)
@@ -59,4 +59,27 @@
       <origin xyz="0.0 0.0 0.0" rpy="0.0 0.0 0.0"/>
     </joint>
+    <!-- ppr -->
+    <!-- fake joint -->
+    <!-- <link name="ppr_fake_link1"/>
+    <link name="ppr_fake_link2"/>
+    <link name="ppr_fake_link3"/>
+    <joint name="motor1" type="prismatic">
+          <parent link="$(arg ur_prefix)wrist_3_link"/>
+          <child link="ppr_fake_link1"/>
+          <axis xyz="0 0 1"/>
+          <limit lower="0" upper="0.027" velocity="0.01" effort="1000.0"/>
+    </joint>
+    <joint name="motor2" type="prismatic">
+          <parent link="$(arg ur_prefix)wrist_3_link"/>
+          <child link="ppr_fake_link2"/>
+          <axis xyz="0 0 1"/>
+          <limit lower="0" upper="0.027" velocity="0.01" effort="1000.0"/>
+    </joint>
+    <joint name="motor3" type="prismatic">
+          <parent link="$(arg ur_prefix)wrist_3_link"/>
+          <child link="ppr_fake_link3"/>
+          <axis xyz="0 0 1"/>
+          <limit lower="0" upper="0.027" velocity="0.01" effort="1000.0"/>
+    </joint> -->
   </xacro:if>
   <!-- IMU -->
